File: Xibidi_calculate/Xibidi_calculate.kicad_sch (KiCad schematic)
At the start: 62 parts, among them J1 USB_C_Receptacle_PowerOnly_6P, SW13 Switch, SW14 Switch, SW15 Switch, SW16 Switch, SW17 Switch, SW18 Switch, SW19 Switch, SW20 Switch, U1 AMS1117-3.3, U11 74LVC2G32, U18 74LVC2G08, U2 74LVC2G86, U20 74LVC2G08, U22 74LVC2G08, U24 74LVC2G08, U4 74LVC2G86, U6 74LVC2G86, U8 74LVC2G86, U9 74LVC2G32

Commit message: files underwent mitosis, should be good still
Connections:
- net at D1.1 (K): now also R25.1; no longer R5.1
- net at D2.1 (K): now also R24.1; no longer R14.1
- net at D4.1 (K): now also R14.1; no longer R24.1
- net at D5.1 (K): now also R5.1; no longer R25.1
Other:
- moved on the sheet: C5, C6, C7, C8, R14, R23, R24, R25, R5
